File: eda/g0dzilla_vs/g0dzilla_vs_rear.kicad_pcb (KiCad board)
At the start: 2 copper layers, 132.2 x 156.8 mm, 6 parts

Commit message: rear pcb with crypto added
Parts:
- added G***: LOGO, 0_alt_bier:logo-alt_bier-900dpi-10x25mm-back, F.Cu at (69.7, 107.0)
- added silk_back_rear: Back Silk, 0_badge:g0dzilla_vs_rear_silk_b, F.Cu at (110.0, 110.0)
