File: eda/g0dzilla_vs/g0dzilla_vs.kicad_sch (KiCad schematic)
At the start: 0 parts

Commit message: middle pcb work
Parts:
- added BT1: Battery_Lipo, 0_local:Battery_Connector_back, symbol 0_local:Battery_Lipo
- added C10, C11, C12, C13, C20, C21, C22, C23: C_Disc_D3, 0_local:C_Disc_D3_back, symbol 0_local:C_Disc_D3
- added D1, D2, D3, D4, D5, D6: LED_3mm, 0_local:LED_D3.0mm-2-std_back, symbol 0_local:LED_THT_3mm
- added D10, D11, D12, D13, D20, D21, D22, D23: LED_WS2812D_5mm, 0_local:LED_D5.0mm-4_WS2812D_2024_back, symbol 0_local:LED_WS2812D_THT_5mm
- added J1: Battery_Conn, 0_local:Battery_Connector_back, symbol 0_local:Battery_Conn
- added J2, J3, J4, J5: 01x02, 0_local:Conn_Pin_Header_Male_Horiz_Back_1x02_Pitch2.54mm, symbol 0_local:Conn_01x02
- added JSAO1, JSAO2, JSAO3, JSAO4: Conn_02x03_SAO, 0_sao_v169bis:SAOv169-BADGEv2-PO-2x3, symbol 0_local:Conn_02x03_SAO
- added R1, R10, R2, R20, R3, R4, R5, R6: 47R_6.3mm, 0_local:R_Axial_DIN0207_L6.3_D2.5_P7.62_Horiz_back, symbol 0_local:R_Axial_Z_L6.3
- added SW1: SW_SPDT_SS12D00G, 0_local:SW_SPDT_Slide_SS12D00G-1P2T_3pin_back, symbol 0_local:SW_SPDT_SS12D00G
- added TCH1, TCH2, TCH3, TCH4: SYM_Touch_lg, symbol 0_local:SYM_Touch_lg
- added U1: ESP32-WEMOS-LOLIN32-LITE, 0_local:ESP32_WEMOS_LOLIN32_LITE_back, symbol 0_local:ESP32-WEMOS-LOLIN32-LITE
Connections:
- new net: D20.4 (DIN), R20.1
- new net: D6.1 (K), R6.1
- new net: D1.1 (K), R1.1
- new net: D10.4 (DIN), R10.1
- new net: BT1.1 (Pin_1), SW1.2 (B)
- new net: D2.1 (K), R2.1
- new net: D3.1 (K), R3.1
- new net: D5.1 (K), R5.1
- new net: D4.1 (K), R4.1
- new net +3.3V: C10.1, C11.1, C12.1, C13.1, C20.1, C21.1, C22.1, C23.1, D10.2 (VDD), D11.2 (VDD), D12.2 (VDD), D13.2 (VDD), D20.2 (VDD), D21.2 (VDD), D22.2 (VDD), D23.2 (VDD), JSAO1.1 (Pin_1), JSAO2.1 (Pin_1), U1.3V3 (3v3)
- new net 13: TCH4.1, U1.13 (GPIO13/TCH4)
- new net 14: D3.2 (A), U1.14 (GPIO14/TCH6)
- new net 15: TCH3.1, U1.15 (GPIO15/TCH3)
- new net 16: R20.2, U1.16 (GPIO16)
- new net 17: R10.2, U1.17 (GPIO17)
- new net 2: TCH2.1, U1.2 (GPIO2/TCH2)
- new net 25: D6.2 (A), U1.25 (GPIO25)
- new net 26: D5.2 (A), U1.26 (GPIO26)
- new net 27: D4.2 (A), U1.27 (GPIO27/TCH7)
- new net 32: D2.2 (A), U1.32 (GPIO32/TCH9)
- new net 33: D1.2 (A), U1.33 (GPIO33/TCH8)
- new net 4: TCH1.1, U1.4 (GPIO4/TCH0)
- new net D10: D10.1 (DOUT), D11.4 (DIN)
- new net D11: D11.1 (DOUT), D12.4 (DIN)
- new net D12: D12.1 (DOUT), D13.4 (DIN)
- new net D20: D20.1 (DOUT), D21.4 (DIN)
- new net D21: D21.1 (DOUT), D22.4 (DIN)
- new net D22: D22.1 (DOUT), D23.4 (DIN)
- new net GBAT: BT1.2 (Pin_2), J1.2 (Pin_2)
- new net GND: C10.2, C11.2, C12.2, C13.2, C20.2, C21.2, C22.2, C23.2, D10.3 (GND), D11.3 (GND), D12.3 (GND), D13.3 (GND), D20.3 (GND), D21.3 (GND), D22.3 (GND), D23.3 (GND), J2.1 (Pin_1), J2.2 (Pin_2), J3.1 (Pin_1), J3.2 (Pin_2), J4.1 (Pin_1), J4.2 (Pin_2), J5.1 (Pin_1), J5.2 (Pin_2), JSAO1.2 (Pin_2), JSAO2.2 (Pin_2), R1.2, R2.2, R3.2, R4.2, R5.2, R6.2, U1.GND
- new net VBAT: J1.1 (Pin_1), SW1.1 (A)
- no-connect marks 0 -> 35
Other:
- note added: "-- Battery Holder -- Four 1x2 right angle header pins and rubber bands between them hold the Lipo Battery in place"
- note added: "-- SAO Storage -- Two 2x3 SAO connectors which are NOT ELECTRICALLY CONNECTED for storing addons on back of the badge when not in use on front of badge"
- note added: "Addon Connectors SAOs"
- note added: "Addressable LEDs"
- note added: "Capacitive Touch"
- note added: "Mechanical"
- note added: "Power"
- note added: "Traditional 2-Pin LEDs"
- note added: "VBAT & GBAT + -"
- note added: "WARNING: JST-PH connector wired reverse polarity from many cables Black wire might go to + & red to - It depends on cable pinout so... DOUBLE CHECK BEFORE CONNECTING!"
- note added: "|- Input ONLY -|"
- company: (none) -> Crafted by @alt_bier a.k.a. Richard Gowen and his Badge Team
- title: (none) -> G0dzilla_VS

Commit message: middle pcb work
Parts:
- added D7, D8: LED_3mm, 0_local:LED_D3.0mm-2-std_back, symbol 0_local:LED_THT_3mm
- added R7, R8: 47R_6.3mm, 0_local:R_Axial_DIN0207_L6.3_D2.5_P7.62_Horiz_back, symbol 0_local:R_Axial_Z_L6.3
- D1, D2, D3, D4, D5: footprint 0_local:LED_D3.0mm-2-std_back -> 0_local:LED_D3.0mm-2-std_front; Color Blue -> White
- D10, D11, D12, D13, D20, D21, D22, D23: footprint 0_local:LED_D5.0mm-4_WS2812D_2024_back -> 0_local:LED_D5.0mm-4_WS2812D_2024_front
- D6: Color Blue -> White
- JSAO1, JSAO2: footprint 0_sao_v169bis:SAOv169-BADGEv2-PO-2x3 -> 0_sao_v169bis:SAOv169-BADGEv3-PO-minF-2x3
- JSAO3, JSAO4: footprint 0_sao_v169bis:SAOv169-BADGEv2-PO-2x3 -> 0_sao_v169bis:SAOv169-BADGEv3-PO-minB-2x3
Connections:
- net 14: now also D4.2 (A); no longer D3.2 (A)
- net 25: now also D2.2 (A); no longer D6.2 (A)
- net 27: now also D3.2 (A); no longer D4.2 (A)
- net 32: now also D1.2 (A); no longer D2.2 (A)
- net 33: now also D6.2 (A); no longer D1.2 (A)
- net GND: now also R7.2, R8.2
- net 35: now reaches JSAO2.6 (Pin_6)
- net 35: now also U1.35 (GPIO35)
- net 34: now reaches JSAO1.6 (Pin_6)
- net 34: now also U1.34 (GPIO34)
- net 12: now reaches U1.12 (GPIO12/TCH5)
- net 12: now also D7.2 (A)
- net 5: now reaches U1.5 (GPIO5)
- net 5: now also D8.2 (A)
- new net: D8.1 (K), R8.1
- new net: D7.1 (K), R7.1
- no-connect marks 35 -> 29
Other:
- moved on the sheet: D1, D2, D3, D4, D5, D6, JSAO1, JSAO2, R1, R2, R3, R4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

Commit message: pcb updates
Parts:
- added R31, R32: 100K_6.3mm, 0_local:R_Axial_DIN0207_L6.3_D2.5_P7.62_Horiz_back, symbol 0_local:R_Axial_Z_L6.3
Connections:
- net 34: now also R31.1
- net 35: now also R32.1
- net GND: now also R31.2, R32.2
Other:
- note added: "Addon Connectors - SAOs"
- note removed: "Addon Connectors SAOs"
- moved on the sheet: BT1, C10, C11, C12, C13, C20, C21, C22, C23, D1, D10, D11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
