File: eda/g0dzilla_vs/g0dzilla_vs_sao1.kicad_sch (KiCad schematic)
At the start: 24 parts

Commit message: final edits before prototype
Parts:
- D1, D2, D21, D22, D31, D32, D41, D42: footprint 0_local:LED_D3.0mm-2-std_front -> 0_local:LED_D3.0mm-2-std_back
- JSAO1, JSAO2, JSAO3, JSAO4: footprint 0_sao_v169bis:SAOv169-BADGEv3-PO-minF-2x3 -> 0_sao_v169bis:SAOv169-SAOv3-2x3
- R33: value 220K_6.3mm -> 100K_6.3mm
- R43: value 100K_6.3mm -> 220K_6.3mm
Connections:
- net +3.3V: no longer D21.2 (A), D22.2 (A), D31.2 (A), D32.2 (A), D41.2 (A), D42.2 (A), JSAO2.1 (Pin_1), JSAO3.1 (Pin_1), JSAO4.1 (Pin_1), R23.2, R33.2, R43.2
- net GND: no longer JSAO2.2 (Pin_2), JSAO3.2 (Pin_2), JSAO4.2 (Pin_2), R21.2, R22.2, R31.2, R32.2, R41.2, R42.2
- new net +3.3V1: D21.2 (A), D22.2 (A), JSAO2.1 (Pin_1), R23.2
- new net +3.3V2: D31.2 (A), D32.2 (A), JSAO3.1 (Pin_1), R33.2
- new net +3.3V3: D41.2 (A), D42.2 (A), JSAO4.1 (Pin_1), R43.2
- new net GND1: JSAO2.2 (Pin_2), R21.2, R22.2
- new net GND2: JSAO3.2 (Pin_2), R31.2, R32.2
- new net GND3: JSAO4.2 (Pin_2), R41.2, R42.2
Other:
- note added: "NOTE: SAO Pin 6 GPIO is used to provide a specific voltage to the badge so that the badge can read this to tell which SAO (monster) is plugged into the badge. 10K = 3V = Mothra 47K = 2.25V = King Ghidorah 100K = 1.65V = Rodan 220K = 1.03V = Hedorah"
- note removed: "NOTE: SAO Pin 6 GPIO is used to provide a specific voltage to the badge so that the badge can read this to tell which SAO (monster) is plugged into the badge. 10K = 3V = Mothra 47K = 2.25V = King Ghidorah 100K = 1.65V = Hedorah 220K = 1.03V = Rodan"
